File: CH224Core/ch224core.kicad_pcb (KiCad board)
At the start: 2 copper layers, 15 x 9.9 mm, 6 parts, among them J1 CH224K, J2 Conn_02x04_Counter_Clockwise, J3 USB4105-GF-A, J4 Conn_01x01

Commit message: update CH224Core PCB
Routing:
- net GND: track 3.22 -> 11.8 mm
Other:
- board text added: "CFG1"
- board text added: "CFG2"
- board text added: "CFG3"
- board text added: "GND"
- board text added: "VBUS"
- board text added: "VDD"
Changed lines of the file:
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@@
   (general
     (thickness 1.6)
-    (drawings 5)
-    (tracks 142)
+    (drawings 18)
+    (tracks 159)
     (zones 0)
     (modules 6)
@@
     (42 Eco1.User user)
     (43 Eco2.User user)
-    (44 Edge.Cuts user)
+    (44 Edge.Cuts user hide)
     (45 Margin user)
     (46 B.CrtYd user hide)
@@
   )
   (setup
-    (last_trace_width 1)
+    (last_trace_width 0.25)
     (user_trace_width 0.3)
     (user_trace_width 0.45)
@@
     (tags resistor)
     (attr smd)
-    (fp_text reference R1 (at 0 -1.3335 270 unlocked) (layer B.SilkS)
+    (fp_text reference R1 (at 0 -1.2065 270 unlocked) (layer B.SilkS)
       (effects (font (size 1 1) (thickness 0.15)) (justify mirror))
     )
     (fp_text value 10k (at 0 -1.43 90) (layer B.Fab)
       (effects (font (size 1 1) (thickness 0.15)) (justify mirror))
-    )
-    (fp_text user %R (at 0 0 90) (layer B.Fab)
-      (effects (font (size 0.4 0.4) (thickness 0.06)) (justify mirror))
     )
     (fp_line (start -0.8 -0.4) (end -0.8 0.4) (layer B.Fab) (width 0.1))
@@
     (fp_line (start 1.48 0.73) (end 1.48 -0.73) (layer B.CrtYd) (width 0.05))
     (fp_line (start 1.48 -0.73) (end -1.48 -0.73) (layer B.CrtYd) (width 0.05))
+    (fp_text user %R (at 0 0 90) (layer B.Fab)
+      (effects (font (size 0.4 0.4) (thickness 0.06)) (justify mirror))
+    )
     (pad 2 smd roundrect (at 0.7875 0 90) (size 0.875 0.95) (layers B.Cu B.Paste B.Mask) (roundrect_rratio 0.25)
       (net 14 "Net-(J1-Pad8)"))
@@
     (tags capacitor)
     (attr smd)
-    (fp_text reference C1 (at -1.0795 1.3335 270) (layer B.SilkS)
+    (fp_text reference C1 (at -1.0795 1.2065 270) (layer B.SilkS)
       (effects (font (size 1 1) (thickness 0.15)) (justify mirror))
     )
     (fp_text value 1u (at 0 -1.43 270) (layer B.Fab)
       (effects (font (size 1 1) (thickness 0.15)) (justify mirror))
-    )
-    (fp_text user %R (at 0 0 270) (layer B.Fab)
-      (effects (font (size 0.4 0.4) (thickness 0.06)) (justify mirror))
     )
     (fp_line (start -0.8 -0.4) (end -0.8 0.4) (layer B.Fab) (width 0.1))
@@
     (fp_line (start 1.48 0.73) (end 1.48 -0.73) (layer B.CrtYd) (width 0.05))
     (fp_line (start 1.48 -0.73) (end -1.48 -0.73) (layer B.CrtYd) (width 0.05))
+    (fp_text user %R (at 0 0 270) (layer B.Fab)
+      (effects (font (size 0.4 0.4) (thickness 0.06)) (justify mirror))
+    )
     (pad 2 smd roundrect (at 0.7875 0 90) (size 0.875 0.95) (layers B.Cu B.Paste B.Mask) (roundrect_rratio 0.25)
       (net 11 GND))
@@
     (pad 10 smd rect (at -2 2.75) (size 0.45 0.81) (layers B.SilkS)
       (net 10 /PG))
+  )
+  (gr_poly (pts (xy 141.732 87.63) (xy 141.2875 87.63) (xy 141.2875 86.8045) (xy 141.732 86.8045)) (layer B.SilkS) (width 0.1))
+  (gr_line (start 138.8745 87.757) (end 138.8745 81.153) (layer Dwgs.User) (width 0.15))
+  (gr_line (start 148.1455 87.757) (end 138.8745 87.757) (layer Dwgs.User) (width 0.15))
+  (gr_line (start 148.1455 81.153) (end 148.1455 87.757) (layer Dwgs.User) (width 0.15))
+  (gr_line (start 138.8745 81.153) (end 148.1455 81.153) (layer Dwgs.User) (width 0.15))
+  (gr_text VDD (at 148.7805 88.265 90) (layer B.SilkS)
+    (effects (font (size 0.6 0.6) (thickness 0.12)) (justify mirror))
+  )
+  (gr_text CFG3 (at 148.7805 85.725 90) (layer B.SilkS)
+    (effects (font (size 0.6 0.6) (thickness 0.12)) (justify mirror))
+  )
+  (gr_text CFG2 (at 148.7805 83.185 90) (layer B.SilkS)
+    (effects (font (size 0.6 0.6) (thickness 0.12)) (justify mirror))
+  )
+  (gr_text CFG1 (at 148.7805 80.645 90) (layer B.SilkS)
+    (effects (font (size 0.6 0.6) (thickness 0.12)) (justify mirror))
+  )
+  (gr_text GND (at 138.2395 83.185 270) (layer B.SilkS)
+    (effects (font (size 0.6 0.6) (thickness 0.12)) (justify mirror))
+  )
+  (gr_text GND (at 138.2395 80.645 270) (layer B.SilkS)
+    (effects (font (size 0.6 0.6) (thickness 0.12)) (justify mirror))
+  )
+  (gr_text VBUS (at 138.2395 88.265 270) (layer B.SilkS)
+    (effects (font (size 0.6 0.6) (thickness 0.12)) (justify mirror))
+  )
+  (gr_text VBUS (at 138.2395 85.725 270) (layer B.SilkS)
+    (effects (font (size 0.6 0.6) (thickness 0.12)) (justify mirror))
   )
   (gr_poly (pts (xy 141.4145 88.4555) (xy 143.002 88.4555) (xy 143.002 88.8365) (xy 144.5895 88.8365) (xy 144.5895 88.4555) (xy 145.6055 88.4555) (xy 145.6055 88.265) (xy 146.2405 88.265) (xy 146.2405 89.408) (xy 140.7795 89.408) (xy 140.7795 88.265) (xy 141.4145 88.265)) (layer F.Mask) (width 0.1))
@@
   (segment (start 144.76 86.617876) (end 144.930606 86.44727) (width 0.3) (layer F.Cu) (net 4))
   (segment (start 144.76 87.686) (end 144.76 86.617876) (width 0.3) (layer F.Cu) (net 4))
-  (segment (start 148.834999 84.699999) (end 149.86 85.725) (width 0.45) (layer B.Cu) (net 5))
+  (segment (start 148.7805 84.6455) (end 149.86 85.725) (width 0.45) (layer B.Cu) (net 5))
   (segment (start 143.51 81.28) (end 144.017999 80.772001) (width 0.45) (layer B.Cu) (net 5))
-  (segment (start 147.543747 80.772001) (end 148.834999 82.063253) (width 0.45) (layer B.Cu) (net 5))
   (segment (start 144.017999 80.772001) (end 147.543747 80.772001) (width 0.45) (layer B.Cu) (net 5))
   (segment (start 143.51 81.705) (end 143.51 81.28) (width 0.45) (layer B.Cu) (net 5))
-  (segment (start 148.834999 82.063253) (end 148.834999 84.699999) (width 0.45) (layer B.Cu) (net 5))
+  (segment (start 147.543747 80.772001) (end 148.7805 82.008754) (width 0.45) (layer B.Cu) (net 5))
+  (segment (start 148.7805 82.008754) (end 148.7805 84.6455) (width 0.45) (layer B.Cu) (net 5))
   (segment (start 141.11 87.686) (end 141.11 88.442504) (width 0.3) (layer F.Cu) (net 6))
-  (via (at 141.11 88.442504) (size 0.6) (drill 0.4) (layers F.Cu B.Cu) (net 6))
+  (via (at 141.11 88.9635) (size 0.6) (drill 0.4) (layers F.Cu B.Cu) (net 6))
   (segment (start 145.91 87.686) (end 145.91 88.442492) (width 0.3) (layer F.Cu) (net 6))
-  (via (at 145.91 88.442492) (size 0.6) (drill 0.4) (layers F.Cu B.Cu) (net 6))
+  (via (at 145.91 88.9635) (size 0.6) (drill 0.4) (layers F.Cu B.Cu) (net 6))
   (segment (start 145.91 88.4685) (end 145.91 88.442492) (width 0.3) (layer F.Cu) (net 6))
   (segment (start 141.11 88.442504) (end 141.11 88.4685) (width 0.3) (layer F.Cu) (net 6))
   (segment (start 141.11 88.4685) (end 141.63675 88.99525) (width 0.3) (layer F.Cu) (net 6))
   (segment (start 141.63675 88.99525) (end 141.790989 89.149489) (width 0.3) (layer F.Cu) (net 6))
-  (via (at 141.63675 88.99525) (size 0.6) (drill 0.4) (layers F.Cu B.Cu) (net 6))
+  (via (at 141.9225 88.99525) (size 0.6) (drill 0.4) (layers F.Cu B.Cu) (net 6))
   (segment (start 137.16 85.725) (end 136.4615 85.0265) (width 0.25) (layer B.Cu) (net 6))
   (segment (start 136.4615 85.0265) (end 138.303 85.0265) (width 0.25) (layer B.Cu) (net 6))
@@
   (segment (start 145.229011 89.149489) (end 145.38325 88.99525) (width 0.3) (layer F.Cu) (net 6))
   (segment (start 141.790989 89.149489) (end 145.229011 89.149489) (width 0.3) (layer F.Cu) (net 6))
-  (via (at 145.38325 88.99525) (size 0.6) (drill 0.4) (layers F.Cu B.Cu) (net 6))
+  (via (at 145.0975 88.99525) (size 0.6) (drill 0.4) (layers F.Cu B.Cu) (net 6))
   (segment (start 141.11 87.686) (end 141.11 87.236) (width 0.3) (layer F.Cu) (net 6))
   (segment (start 141.11 87.686) (end 141.11 87.120002) (width 0.3) (layer F.Cu) (net 6))
@@
   (segment (start 147.83 87.111) (end 147.83 86.5525) (width 1) (layer B.Cu) (net 11))
   (segment (start 147.83 86.616) (end 147.32 86.106) (width 1) (layer B.Cu) (net 11))
+  (segment (start 139.19 87.111) (end 139.308 87.111) (width 1) (layer F.Cu) (net 11))
+  (segment (start 139.883 87.686) (end 140.109999 87.686) (width 1) (layer F.Cu) (net 11))
+  (segment (start 139.308 87.111) (end 139.883 87.686) (width 1) (layer F.Cu) (net 11))
+  (segment (start 139.19 87.111) (end 139.19 86.5485) (width 0.25) (layer F.Cu) (net 11))
+  (segment (start 139.19 87.111) (end 139.19 86.866) (width 0.25) (layer F.Cu) (net 11))
+  (segment (start 139.19 86.866) (end 138.811 86.487) (width 0.25) (layer F.Cu) (net 11))
+  (segment (start 138.811 86.487) (end 138.811 85.7885) (width 0.25) (layer F.Cu) (net 11))
+  (segment (start 139.19 86.358) (end 139.0015 86.1695) (width 0.25) (layer F.Cu) (net 11))
+  (segment (start 139.19 87.111) (end 139.19 86.358) (width 0.3) (layer F.Cu) (net 11))
+  (segment (start 138.938 86.859) (end 139.19 87.111) (width 0.3) (layer F.Cu) (net 11))
+  (segment (start 138.938 85.7885) (end 138.938 86.859) (width 0.3) (layer F.Cu) (net 11))
+  (segment (start 139.19 87.111) (end 139.19 86.485) (width 0.3) (layer B.Cu) (net 11))
+  (segment (start 139.19 86.485) (end 138.938 86.233) (width 0.3) (layer B.Cu) (net 11))
+  (segment (start 138.938 86.233) (end 138.938 85.7885) (width 0.3) (layer B.Cu) (net 11))
+  (segment (start 139.19 87.111) (end 139.19 86.739) (width 0.25) (layer B.Cu) (net 11))
+  (segment (start 139.19 86.739) (end 138.811 86.36) (width 0.25) (layer B.Cu) (net 11))
+  (segment (start 138.811 86.36) (end 138.811 85.7885) (width 0.25) (layer B.Cu) (net 11))
   (segment (start 143.51 87.205) (end 143.51 86.4235) (width 0.3) (layer B.Cu) (net 14))
   (via (at 143.129 86.0425) (size 0.5) (drill 0.3) (layers F.Cu B.Cu) (net 14))
