File: bbSink/ch224base.sch (KiCad schematic (older format))
At the start: 37 parts, among them IC1 NCP1117, J1 Conn_02x04_Counter_Clockwise, J2 Conn_01x02, J3 Conn_02x04_Counter_Clockwise, SW1 SW_DIP_x01, SW2 SW_DIP_x01, SW3 SW_DIP_x01, SW4 SW_DIP_x01, SW5 SW_DIP_x01, U1 74HC32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

Commit message: update docs
Parts:
- C1: value 1u -> NC
- R4: value 51k -> 15k
- R5: value 160k -> 47k
- U2: symbol ch224base-rescue:MPM3620GQV-Z-2021-04-10_02-29-46-ch224base-rescue-ch224base-rescue -> 2021-04-10_02-29-46:MPM3620GQV-Z
Changed lines of the file:
@@
 VBUS
 $Comp
-L ch224base-rescue:MPM3620GQV-Z-2021-04-10_02-29-46-ch224base-rescue-ch224base-rescue U2
+L 2021-04-10_02-29-46:MPM3620GQV-Z U2
 U 1 1 60714179
 P 8050 5000
@@
 P 2050 6000
 F 0 "C1" V 1798 6000 50  0000 C CNN
-F 1 "1u" V 1889 6000 50  0000 C CNN
+F 1 "NC" V 1889 6000 50  0000 C CNN
 F 2 "Capacitor_SMD:C_0603_1608Metric" H 2088 5850 50  0001 C CNN
 F 3 "~" H 2050 6000 50  0001 C CNN
@@
 P 7900 5000
 F 0 "R4" H 7970 5046 50  0000 L CNN
-F 1 "51k" H 7970 4955 50  0000 L CNN
+F 1 "15k" H 7970 4955 50  0000 L CNN
 F 2 "Resistor_SMD:R_0603_1608Metric" V 7830 5000 50  0001 C CNN
 F 3 "~" H 7900 5000 50  0001 C CNN
@@
 P 8050 4800
 F 0 "R5" H 8120 4846 50  0000 L CNN
-F 1 "160k" H 8120 4755 50  0000 L CNN
+F 1 "47k" H 8120 4755 50  0000 L CNN
 F 2 "Resistor_SMD:R_0603_1608Metric" V 7980 4800 50  0001 C CNN
 F 3 "~" H 8050 4800 50  0001 C CNN
